Commit message: urdf updated

File: src/HACK13/description/ackermann.urdf.xacro (robot description, xacro)
@@ -50,5 +50,5 @@
     </visual>
 </link>
-<joint name="joint_name" type="prismatic">
+<joint name="rack_joint" type="prismatic">
     <origin xyz="-0.0315 0.0 0.0"/>
     <parent link="base_link"/>
@@ -85,3 +85,18 @@
     <axis xyz="0.0 0.0 1.0"/>
 </joint>
+<link name="pinion">
+    <visual>
+        <origin xyz="0.0 0.0 0.0"/>
+        <geometry>
+            <cylinder radius="0.0381" length="0.0254"/>
+        </geometry>
+    </visual>
+</link>
+<joint name="pinion_joint" type="revolute">
+    <origin xyz="-0.0315 0.0 0.04445" rpy="0.0 ${pi/2} 0.0"/>
+    <parent link="base_link"/>
+    <child link="pinion"/>
+    <axis xyz="0.0 0.0 1.0"/>
+    <limit lower="-1.586" upper="1.586" effort="0.0" velocity="0.0"/>
+</joint>
 </robot>

Commit message: working?

File: src/HACK13/description/ackermann.urdf.xacro (robot description, xacro)
@@ -1,4 +1,8 @@
 <?xml version="1.0"?>
 <robot xmlns:xacro="http://www.ros.org/wiki/xacro" name="sarah7">
+  <!-- ===== Macros ===== -->
+  <xacro:include filename="macros/materials.xacro"/>
+  <xacro:include filename="macros/inertials.xacro"/>
+  <xacro:include filename="macros/components.xacro"/>
 <link name="base_link"/>
 <link name="frame">
@@ -91,4 +95,5 @@
             <cylinder radius="0.0381" length="0.0254"/>
         </geometry>
+      <material name="black"/>
     </visual>
 </link>
@@ -100,3 +105,75 @@
     <limit lower="-1.586" upper="1.586" effort="0.0" velocity="0.0"/>
 </joint>
+<link name="lf_wheel">
+  <visual>
+    <geometry>
+      <cylinder radius="0.1524" length="0.0762"/>
+    </geometry>
+      <material name="blue"/>
+  </visual>
+</link>
+<link name="rf_wheel">
+  <visual>
+    <geometry>
+      <cylinder radius="0.1524" length="0.0762"/>
+    </geometry>
+      <material name="blue"/>
+  </visual>
+</link>
+<joint name="lf_wjoint" type="fixed">
+  <parent link="left_steering_arm"/>
+  <child link="lf_wheel"/>
+  <origin xyz="0.1 0.0 0.0" rpy="0.0 -1.57 0.0"/>
+</joint>
+<joint name="rf_wjoint" type="fixed">
+  <parent link="right_steering_arm"/>
+  <child link="rf_wheel"/>
+  <origin xyz="0.1 0.0 0.0" rpy="0.0 -1.57 0.0"/>
+</joint>
+<link name="diff"></link>
+<joint name="diff_j" type="fixed">
+  <parent link="base_link"/>
+  <child link="diff"/>
+  <origin xyz="-0.9144 0.0 0.0"/>
+</joint>
+<link name="lr_wheel">
+  <visual>
+    <geometry>
+      <cylinder radius="0.1524" length="0.0762"/>
+    </geometry>
+      <material name="blue"/>
+  </visual>
+</link>
+<link name="rr_wheel">
+  <visual>
+    <geometry>
+      <cylinder radius="0.1524" length="0.0762"/>
+    </geometry>
+      <material name="blue"/>
+  </visual>
+</link>
+<joint name="lr_wjoint" type="fixed">
+  <parent link="diff"/>
+  <child link="lr_wheel"/>
+  <origin xyz="0.0 0.4048 0.0" rpy="-1.57 0.0 0.0"/>
+</joint>
+<joint name="rr_wjoint" type="fixed">
+  <parent link="diff"/>
+  <child link="rr_wheel"/>
+  <origin xyz="0.0 -0.4048 0.0" rpy="-1.57 0.0 0.0"/>
+</joint>
+  <!-- ===== CHASSIS ===== -->
+  <link name="chassis_link">
+    <visual>
+      <geometry>
+        <box size="0.9144 0.6096 0.1524"/>
+      </geometry>
+      <material name="white"/>
+    </visual>
+  </link>
+  <joint name="chassis_joint" type="fixed">
+    <parent link="base_link"/>
+    <child link="chassis_link"/>
+    <origin xyz="-0.4572 0.0 0.0762"/>
+  </joint>
 </robot>

Commit message: ahh

File: src/HACK13/description/ackermann.urdf.xacro (robot description, xacro)
@@ -1,4 +1,6 @@
 <?xml version="1.0"?>
 <robot xmlns:xacro="http://www.ros.org/wiki/xacro" name="sarah7">
+  <!-- ===== Macros ===== -->
+  <xacro:include filename="macros/materials.xacro"/>
 <link name="base_link"/>
 <link name="frame">
@@ -91,4 +93,5 @@
             <cylinder radius="0.0381" length="0.0254"/>
         </geometry>
+      <material name="black"/>
     </visual>
 </link>
@@ -100,3 +103,75 @@
     <limit lower="-1.586" upper="1.586" effort="0.0" velocity="0.0"/>
 </joint>
+<link name="lf_wheel">
+  <visual>
+    <geometry>
+      <cylinder radius="0.1524" length="0.0762"/>
+    </geometry>
+      <material name="blue"/>
+  </visual>
+</link>
+<link name="rf_wheel">
+  <visual>
+    <geometry>
+      <cylinder radius="0.1524" length="0.0762"/>
+    </geometry>
+      <material name="blue"/>
+  </visual>
+</link>
+<joint name="lf_wjoint" type="fixed">
+  <parent link="left_steering_arm"/>
+  <child link="lf_wheel"/>
+  <origin xyz="0.1 0.0 0.0" rpy="0.0 -1.57 0.0"/>
+</joint>
+<joint name="rf_wjoint" type="fixed">
+  <parent link="right_steering_arm"/>
+  <child link="rf_wheel"/>
+  <origin xyz="0.1 0.0 0.0" rpy="0.0 -1.57 0.0"/>
+</joint>
+<link name="diff"></link>
+<joint name="diff_j" type="fixed">
+  <parent link="base_link"/>
+  <child link="diff"/>
+  <origin xyz="-0.9144 0.0 0.0"/>
+</joint>
+<link name="lr_wheel">
+  <visual>
+    <geometry>
+      <cylinder radius="0.1524" length="0.0762"/>
+    </geometry>
+      <material name="blue"/>
+  </visual>
+</link>
+<link name="rr_wheel">
+  <visual>
+    <geometry>
+      <cylinder radius="0.1524" length="0.0762"/>
+    </geometry>
+      <material name="blue"/>
+  </visual>
+</link>
+<joint name="lr_wjoint" type="fixed">
+  <parent link="diff"/>
+  <child link="lr_wheel"/>
+  <origin xyz="0.0 0.4048 0.0" rpy="-1.57 0.0 0.0"/>
+</joint>
+<joint name="rr_wjoint" type="fixed">
+  <parent link="diff"/>
+  <child link="rr_wheel"/>
+  <origin xyz="0.0 -0.4048 0.0" rpy="-1.57 0.0 0.0"/>
+</joint>
+  <!-- ===== CHASSIS ===== -->
+  <link name="chassis_link">
+    <visual>
+      <geometry>
+        <box size="0.9144 0.6096 0.1524"/>
+      </geometry>
+      <material name="white"/>
+    </visual>
+  </link>
+  <joint name="chassis_joint" type="fixed">
+    <parent link="base_link"/>
+    <child link="chassis_link"/>
+    <origin xyz="-0.4572 0.0 0.0762"/>
+  </joint>
 </robot>
